File: Hardware/PCB/output expander front panel/harp output expander front panel.kicad_pcb (KiCad board)
At the start: 2 copper layers, 133 x 35 mm, 17 parts

Commit message: Updated Gerbers.
Parts:
- added ref1: harp_logo, stepperdriver front panel:harp_logo, F.Cu at (93.6, 118.3)
Other:
- board text removed: "Powered by:"
