File: Hardware/PCB/output expander/IOs.kicad_sch (KiCad schematic)
At the start: 68 parts, among them IC10 SN74LVC1G125DBVT, IC7 SN74LVC1G125DBVT, U1 SN74LVC4245APWR, U2 SN74LVC4245APWR, U3 74HCT125D,653

Commit message: Fixed IC6 MPN and footprint, and U1-2 MPN
Parts:
- BNC0, BNC1, BNC2, BNC3, BNC4: MPN 731000105 -> 0731000105; OEPS Description (none) -> CONNECTOR: BNC JACK 50ohm R/A [0731000105] [TH]
- C27, C28, C29, C30, C31, C32, C40: OEPS Description (none) -> CAPACITOR: SMD CER 0402 100nF 50V ±10% X7R [CGA2B3X7R1H104K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
- C33, C34, C37, C38: OEPS Description (none) -> CAPACITOR: SMD CER 0603 4.7uF 16V ±10% X6S [C1608X6S1C475K0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
- C41, C42, C43, C44, C45, C46, C47, C48, C49, C50: OEPS Description (none) -> CAPACITOR: SMD CER 0402 330pF 50V ±5% C0G [C0402C331J5GAC78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
- IC10, IC7: OEPS Description (none) -> IC: BUFFER NON-INVERT 1CH 3-STATE [SN74LVC1G125DBVT] [SOT-2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
- R10, R11, R12, R13, R14, R15, R16, R17, R19, R38, R43, R46, R47, R56, R57, R58, R59, R60, R61, R62, R63, R64, R65, R66, R67, R9: OEPS Description (none) -> RESISTOR: SMD 0402 10kΩ ±1% 0.063W [CRCW040210K0FKED] [SMD]
- R4, R48, R49, R5, R50, R51, R52, R6, R7, R8: OEPS Description (none) -> RESISTOR: SMD 0603 100Ω ±1% 0.333W [CRCW0603100RFKEAHP] [SM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
- SV1: OEPS Description (none) -> CONNECTOR: HEADER 2.54MM R/A 2x5POS [SBH11-PBPC-D05-RA-BK] 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
- U1, U2: value SN74LVC4245APWR -> SN74LVC8T245DWR; MPN SN74LVC4245APWR -> SN74LVC8T245DWR; OEPS Description (none) -> IC: LEVEL TRANSLATOR 8CH BIDIRECTIONAL [SN74LVC8T245DWR] [2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; OEPSPN OEPS080126 -> OEPS080253
- U3: OEPS Description (none) -> IC: BUFFER NON-INVERT 4CH 3-STATE [74HCT125D,653] [SOIC-14]
Other:
- note removed: "MPN original: 74LVC4245AD,118"
