File: Hardware/PCB/output expander/LEDs & ClockIO.kicad_sch (KiCad schematic)
At the start: 58 parts, among them IC5 TLV70033DDCR, IC6 SI8621BC-B-ISR, IC8 SN74LVC1G125DBVT, IC9 SN74LVC1G125DBVT, T10 BC850C,215, T11 BC850C,215, T12 BC850C,215, T13 BC850C,215, T2 BC850C,215, T3 BC850C,215, T4 BC850C,215, T5 BC850C,215, T6 BC850C,215, T7 BC850C,215, T8 BC850C,215, T9 BC850C,215

Commit message: Fixed IC6 MPN and footprint, and U1-2 MPN
Parts:
- C23, C24: OEPS Description (none) -> CAPACITOR: SMD CER 0603 4.7uF 16V ±10% X6S [C1608X6S1C475K0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
- C25, C26, C35, C36: OEPS Description (none) -> CAPACITOR: SMD CER 0402 100nF 50V ±10% X7R [CGA2B3X7R1H104K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
- CLKIN0, CLKOUT0: OEPS Description (none) -> CONNECTOR: 3.5MM JACK STEREO 90º [35RASMT2BHNTRX] [SMD]
- IC5: OEPS Description (none) -> IC: LDO 3.3V 200mA [TLV70033DDCR] [SOT-23-THIN]
- IC6: value SI8621BC-B-ISR -> SI8610BC-B-IS; footprint Package_SO:SOIC-8_5.3x5.3mm_P1.27mm -> Package_SO:SOIC-8_3.9x4.9mm_P1.27mm; MPN SI8621BC-B-ISR -> SI8610BC-B-ISR; OEPS Description (none) -> IC: DIGITAL ISOLATOR 1WAY [SI8610BC-B-ISR] [8-SOIC]; OEPSPN OEPS080031 -> OEPS080004
- IC8, IC9: OEPS Description (none) -> IC: BUFFER NON-INVERT 1CH 3-STATE [SN74LVC1G125DBVT] [SOT-2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
- LED0, LED1, LED2, LED3, LED4, LED5: OEPS Description (none) -> DIODE: LED DUAL Red 635nm 20mA [569-0111-100F] [TH]
- R2: OEPS Description (none) -> RESISTOR: SMD 0402 10Ω ±5% 0.25W [ERJ-PA2J100X] [SMD]
- R20, R21, R22, R23, R24, R25, R26, R27, R28, R29, R30, R31: OEPS Description (none) -> RESISTOR: SMD 0402 1kΩ ±1% 0.063W [CRCW04021K00FKED] [SMD]
- R3, R54, R55: OEPS Description (none) -> RESISTOR: SMD 0402 10kΩ ±1% 0.063W [CRCW040210K0FKED] [SMD]
- R32, R33, R34, R35, R36, R37, R39, R40, R41, R42, R44, R45: OEPS Description (none) -> RESISTOR: SMD 0402 330Ω ±1% 0.063W [RC0402FR-07330RL] [SMD]
- T10, T11, T12, T13, T2, T3, T4, T5, T6, T7, T8, T9: OEPS Description (none) -> TRANSISTOR: BJT NPN 45V 0.1A [BC850C,215] [SOT-23-3]
