File: Hardware/PCB/output expander/harp expander output.kicad_sch (KiCad schematic)
At the start: 24 parts, among them IC2 USBLC6-2SC6, IC3 FT232RL-REEL, IC4 TLV70033DDCR

Commit message: Fixed IC6 MPN and footprint, and U1-2 MPN
Parts:
- C10, C11, C52: OEPS Description (none) -> CAPACITOR: SMD CER 0603 4.7uF 16V ±10% X6S [C1608X6S1C475K0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
- C12, C3, C5, C7, C9: OEPS Description (none) -> CAPACITOR: SMD CER 0402 100nF 50V ±10% X7R [CGA2B3X7R1H104K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
- C2: OEPS Description (none) -> CAPACITOR: SMD CER 0402 4.7nF 100V ±10% X7R [885012205084] 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
- C39: OEPS Description (none) -> CAPACITOR POL: TH ALUM 100uF 25V ±20% 130mOhm [EEU-FM1E101B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
- C4, C6: OEPS Description (none) -> CAPACITOR: SMD CER 0402 47pF 50V ±5% C0G [04025A470JAT2A] [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
- IC2: OEPS Description (none) -> DIODE: TVS DIODE 5.25VWM 17VC [USBLC6-2SC6] [SOT-23-6]
- IC3: OEPS Description (none) -> IC: USB Interface IC USB to Serial UART (OEPS NP1 073) [FT2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
- IC4: OEPS Description (none) -> IC: LDO 3.3V 200mA [TLV70033DDCR] [SOT-23-THIN]
- L1: OEPS Description (none) -> INDUCTOR: FERRITE BEAD SMD 40Ω 2A 50mΩ [MI0805K400R-10] [08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
- R1, R18: OEPS Description (none) -> RESISTOR: SMD 0402 5.1kΩ ±1% 0.100W [ERJ-2RKF5101X] [SMD]
- R69: OEPS Description (none) -> RESISTOR: SMD 0603 100Ω ±1% 0.333W [CRCW0603100RFKEAHP] [SM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
- USB0: OEPS Description (none) -> CONNECTOR: USB2.0 TYPE C 16P SMD R/A [USB4105-GF-A] [SMD/TH]
